File: LuckFox-RAP-Shield-PCB/LuckFox RAP Shield.kicad_pcb (KiCad board)
At the start: 2 copper layers, 45 x 63.2 mm, 8 parts, among them J1 LuckFox_Pico_Mini_Connector, J2 External_5V_Input_from_Buck_M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, U2 W5500_Ethernet_Module_DNP_on_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

Commit message: Insert logo to PCB
Parts:
- added G***: LOGO, footprints:logo, F.Cu at (134.6, 94.6)
Other:
- board text added: "REV A"
